Commit message: added links transforms and packages from ros2 differential drive tutorials

File: autonomous_waiter_description/src/description/autonomous_waiter_description.urdf (robot description, URDF)
Before this commit: robot autonomous_waiter, 0 links, 0 joints
Links:
- added link base_footprint
- added link base_link; visual box size=${base_length} ${base_width} ${base_height}
- added link front_caster; visual sphere radius=${(wheel_radius+wheel_zoff-(base_height/2))}
Joints:
- added joint base_joint: type fixed, parent base_link, child base_footprint, origin xyz=0.0 0.0 ${-(wheel_radius+wheel_zoff)} rpy=0 0 0
- added joint caster_joint: type fixed, parent base_link, child front_caster, origin xyz=${caster_xoff} 0.0 ${-(base_height/2)} rpy=0 0 0
