Commit message: gazebo config (right before trying to implement with actual robot)

File: autonomous_waiter_description/src/description/ros2_control.xacro (robot description, xacro)
@@ -1,9 +1,9 @@
 <?xml version="1.0"?>
 <robot xmlns:xacro="http://www.ros.org/wiki/xacro">
-    <ros2_control name="GazeboSystem" type="system">
+    <ros2_control name="GazeboSystem" type="actuator">
         <hardware>
-            <plugin>gazebo_ros2_control/GazeboSystem</plugin>
+            <plugin>diff_drive_pico/DiffDrivePico</plugin>
         </hardware>
-        <joint name="left_wheel_joint">
+        <joint name="drivewhl_l_joint">
             <command_interface name="velocity">
                 <param name="min">-10</param>
@@ -13,5 +13,5 @@
             <state_interface name="position"/>
         </joint>
-        <joint name="right_wheel_joint">
+        <joint name="drivewhl_r_joint">
             <command_interface name="velocity">
                 <param name="min">-10</param>
@@ -23,6 +23,6 @@
     </ros2_control>
     <gazebo>
-        <plugin name="gazebo_ros2_control" filename="libgazebo_ros2_control.so">
-            <parameters>$(find articubot_one)/config/my_controllers.yaml</parameters>
+        <plugin name="diff_drive" filename="libgazebo_ros2_control.so">
+            <parameters>$(find autonomous_waiter_description)/config/my_controllers.yaml</parameters>
         </plugin>
     </gazebo>

Commit message: ready to launch?

File: autonomous_waiter_description/src/description/ros2_control.xacro (robot description, xacro)
@@ -1,5 +1,26 @@
 <?xml version="1.0"?>
 <robot xmlns:xacro="http://www.ros.org/wiki/xacro">
-    <ros2_control name="GazeboSystem" type="actuator">
+    <!-- <ros2_control name="GazeboSystem" type="actuator">
+        <hardware>
+            <plugin>diff_drive_pico/DiffDrivePico</plugin>
+        </hardware>
+        <joint name="drivewhl_l_joint">
+            <command_interface name="velocity">
+                <param name="min">-10</param>
+                <param name="max">10</param>
+            </command_interface>
+            <state_interface name="velocity"/>
+            <state_interface name="position"/>
+        </joint>
+        <joint name="drivewhl_r_joint">
+            <command_interface name="velocity">
+                <param name="min">-10</param>
+                <param name="max">10</param>
+            </command_interface>
+            <state_interface name="velocity"/>
+            <state_interface name="position"/>
+        </joint>
+    </ros2_control> -->
+    <ros2_control name="RealRobot" type="actuator">
         <hardware>
             <plugin>diff_drive_pico/DiffDrivePico</plugin>
