Commit message: edited slam and lidar configs and simulation params

File: autonomous_waiter_description/description/autonomous_waiter_description.urdf (robot description, URDF)
Before this commit: robot autonomous_waiter, 3 links, 2 joints
Links:
- added link wheel_l_link; collision cylinder length=${wheel_width} radius=${wheel_radius}; visual cylinder length=${wheel_width} radius=${wheel_radius}
- added link wheel_r_link; collision cylinder length=${wheel_width} radius=${wheel_radius}; visual cylinder length=${wheel_width} radius=${wheel_radius}
Joints:
- added joint wheel_l_joint: type continuous, parent base_link, child wheel_l_link, origin xyz=${1*wheel_xoff} ${1*(base_width/2+wheel_ygap)} ${-wheel_zoff} rpy=0 0 0, axis 0 1 0
- added joint wheel_r_joint: type continuous, parent base_link, child wheel_r_link, origin xyz=${1*wheel_xoff} ${-1*(base_width/2+wheel_ygap)} ${-wheel_zoff} rpy=0 0 0, axis 0 1 0

File: autonomous_waiter_description/description/lidar.xacro (robot description, xacro)
@@ -1,5 +1,5 @@
 <?xml version="1.0"?>
 <robot xmlns:xacro="http://www.ros.org/wiki/xacro">
-  <link name="lidar_link">
+  <link name="laser_frame">
     <inertial>
       <origin xyz="0 0 0" rpy="0 0 0"/>
@@ -22,8 +22,8 @@
   <joint name="lidar_joint" type="fixed">
     <parent link="base_link"/>
-    <child link="lidar_link"/>
+    <child link="laser_frame"/>
     <origin xyz="0 0 0.12" rpy="0 0 0"/>
   </joint>
-  <gazebo reference="lidar_link">
+  <!-- <gazebo reference="lidar_link">
     <sensor name="lidar" type="ray">
       <always_on>true</always_on>
@@ -58,4 +58,4 @@
       </plugin>
     </sensor>
-  </gazebo>
+  </gazebo> -->
 </robot>

File: autonomous_waiter_description/description/ros2_control.xacro (robot description, xacro)
@@ -26,5 +26,5 @@
             <plugin>diff_drive_pico/DiffDrivePico</plugin>
         </hardware>
-        <joint name="drivewhl_l_joint">
+        <joint name="wheel_l_joint">
             <command_interface name="velocity">
                 <param name="min">0</param>
@@ -34,5 +34,5 @@
             <state_interface name="velocity"/>
         </joint>
-        <joint name="drivewhl_r_joint">
+        <joint name="wheel_r_joint">
             <command_interface name="velocity">
                 <param name="min">0</param>
